File: kalckert/force-servo/drawings/arduinoshield.brd (EAGLE design)
At the start: 100 x 80 mm, 36 parts, among them IC1 MCP604P, IC3 7806T, IC5 MCP604P

Commit message: Moved tapometer from its own folder to project folder and added drawings and the CERn hardware licence to the drawings.
Parts:
- removed C3: 330nF, rcl:C025-025X050
- removed C4: 100nF, rcl:C025-025X050
- removed IC3: 7806T, linear:TO220H
- removed SG4: F/QMX, buzzer:F/QMX
- added JP2: (no value), jumper:JP1
Connections:
- removed net N$14: C9.+, IC2.3
- removed net N$20: C10.1, C8.+, IC2.2, R7.2
- net GND: now also JP2.1; no longer C6.2
- net N$3: now also C6.2, JP2.2; no longer C3.2, C4.2, IC3.2
- net VCCSERVO: now also C8.+, IC2.2, R7.2; no longer C4.1, IC3.3
- net VIN: now also C10.1, C9.+, IC2.3; no longer C3.1, IC3.1
Routing:
- net GND: track 180.5 -> 145.4 mm
- net N$3: track 6.77 -> 0.00 mm
- net VIN: track 50.9 -> 44.3 mm
Changed lines of the file:
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@@
 </element>
 <element name="R2" library="pot" package="S64W" value="" x="50.673" y="27.686" rot="R270"/>
-<element name="C3" library="rcl" package="C025-025X050" value="330nF" x="26.035" y="22.86" rot="R90"/>
-<element name="C4" library="rcl" package="C025-025X050" value="100nF" x="26.035" y="28.321" rot="R270"/>
-<element name="IC3" library="linear" package="TO220H" value="7806T" x="11.43" y="25.527" rot="R90"/>
 <element name="IC4" library="linear" package="TO220H" value="" x="11.43" y="13.081" rot="R90"/>
-<element name="SG4" library="buzzer" package="F/QMX" value="F/QMX" x="80.137" y="59.69" rot="R90">
-<attribute name="OC_NEWARK" value="unknown" x="80.137" y="59.69" size="1.778" layer="27" rot="R90" display="off"/>
-<attribute name="MPN" value="" x="80.137" y="59.69" size="1.778" layer="27" rot="R90" display="off"/>
-<attribute name="MF" value="" x="80.137" y="59.69" size="1.778" layer="27" rot="R90" display="off"/>
-<attribute name="OC_FARNELL" value="unknown" x="80.137" y="59.69" size="1.778" layer="27" rot="R90" display="off"/>
-</element>
 <element name="C6" library="resistor" package="C050-025X075" value="10uF" x="21.209" y="2.54" rot="R180"/>
 <element name="R5" library="resistor" package="0207/7" value="82k" x="-1.524" y="-3.937"/>
@@
 <element name="S1" library="switch" package="MS243" value="" x="-14.605" y="-85.471"/>
 <element name="R3" library="resistor" package="0207/7" value="68" x="-13.335" y="-93.98"/>
+<element name="JP2" library="jumper" package="JP1" value="" x="-28.575" y="-92.075"/>
 </elements>
 <signals>
@@
 <wire x1="39.37" y1="20.32" x2="39.37" y2="20.066" width="0.254" layer="16"/>
 <wire x1="21.59" y1="15.24" x2="21.59" y2="15.621" width="0.254" layer="16"/>
-<contactref element="C6" pad="2"/>
-<wire x1="10.16" y1="11.43" x2="19.05" y2="2.54" width="0.254" layer="16"/>
-<wire x1="10.16" y1="31.75" x2="10.16" y2="11.43" width="0.254" layer="16"/>
-<wire x1="8.89" y1="33.02" x2="10.16" y2="31.75" width="0.254" layer="16"/>
-<wire x1="19.05" y1="2.54" x2="18.669" y2="2.54" width="0.254" layer="16"/>
 <contactref element="C7" pad="2"/>
 <contactref element="C5" pad="2"/>
@@
 <contactref element="R4" pad="1"/>
 <contactref element="R3" pad="1"/>
+<contactref element="JP2" pad="1"/>
+<wire x1="-17.145" y1="-93.98" x2="-28.575" y2="-93.345" width="0" layer="19" extent="1-1"/>
 <wire x1="-17.145" y1="-73.025" x2="-17.145" y2="-93.98" width="0" layer="19" extent="1-1"/>
 <wire x1="-17.145" y1="-52.578" x2="-17.145" y2="-73.025" width="0" layer="19" extent="1-1"/>
@@
 <wire x1="-2.413" y1="-17.272" x2="-14.351" y2="-23.622" width="0" layer="19" extent="1-1"/>
 <wire x1="-2.413" y1="-12.7" x2="-2.413" y2="-17.272" width="0" layer="19" extent="1-1"/>
-<wire x1="18.669" y1="2.54" x2="-2.413" y2="-12.7" width="0" layer="19" extent="1-1"/>
-<wire x1="9.271" y1="33.782" x2="8.89" y2="33.02" width="0" layer="19" extent="1-16"/>
+<wire x1="21.59" y1="15.24" x2="-2.413" y2="-12.7" width="0" layer="19" extent="16-16"/>
 </signal>
 <signal name="VCCSERVO">
 <contactref element="SERVOPIN" pad="2"/>
-<contactref element="C4" pad="1"/>
-<contactref element="IC3" pad="3"/>
 <wire x1="24.13" y1="27.94" x2="30.988" y2="34.798" width="0.254" layer="1"/>
 <wire x1="21.59" y1="27.94" x2="24.13" y2="27.94" width="0.254" layer="1"/>
-<wire x1="21.59" y1="27.94" x2="21.59" y2="28.067" width="0.254" layer="1"/>
-<wire x1="24.13" y1="27.94" x2="26.035" y2="29.591" width="0" layer="19" extent="1-1"/>
+<contactref element="R7" pad="2"/>
+<contactref element="IC2" pad="2"/>
+<contactref element="C8" pad="+"/>
+<wire x1="-16.891" y1="-23.622" x2="-9.525" y2="-43.942" width="0" layer="19" extent="1-1"/>
+<wire x1="-12.954" y1="-18.415" x2="-16.891" y2="-23.622" width="0" layer="19" extent="1-1"/>
+<wire x1="21.59" y1="27.94" x2="-12.954" y2="-18.415" width="0" layer="19" extent="1-1"/>
 </signal>
 <signal name="SERVOPWM">
@@
 <signal name="VIN">
 <contactref element="POWERPIN" pad="8"/>
-<contactref element="C3" pad="1"/>
-<contactref element="IC3" pad="1"/>
-<wire x1="21.59" y1="21.59" x2="26.035" y2="21.59" width="0.254" layer="1"/>
-<wire x1="21.59" y1="22.987" x2="21.59" y2="21.59" width="0.254" layer="1"/>
-<wire x1="25.4" y1="21.59" x2="26.035" y2="21.59" width="0.254" layer="16"/>
 <wire x1="39.37" y1="8.89" x2="45.72" y2="2.54" width="0.254" layer="16"/>
 <wire x1="19.05" y1="8.89" x2="39.37" y2="8.89" width="0.254" layer="16"/>
 <wire x1="21.59" y1="22.86" x2="19.05" y2="20.32" width="0.254" layer="16"/>
-<wire x1="21.59" y1="22.86" x2="21.59" y2="22.987" width="0.254" layer="16"/>
 <wire x1="19.05" y1="8.89" x2="19.05" y2="20.32" width="0.254" layer="16"/>
-</signal>
-<signal name="N$3">
-<contactref element="IC3" pad="2"/>
-<wire x1="22.86" y1="26.67" x2="25.4" y2="24.13" width="0.254" layer="1"/>
-<wire x1="21.59" y1="26.67" x2="22.86" y2="26.67" width="0.254" layer="1"/>
-<wire x1="21.59" y1="25.527" x2="21.59" y2="26.67" width="0.254" layer="1"/>
-<wire x1="21.59" y1="25.4" x2="21.59" y2="25.527" width="0.254" layer="1"/>
-<contactref element="C3" pad="2"/>
-<contactref element="C4" pad="2"/>
-<wire x1="25.4" y1="24.13" x2="26.035" y2="24.13" width="0.254" layer="1"/>
-<wire x1="26.035" y1="24.13" x2="26.035" y2="27.051" width="0" layer="19" extent="1-1"/>
+<contactref element="C10" pad="1"/>
+<contactref element="IC2" pad="3"/>
+<contactref element="C9" pad="+"/>
+<wire x1="-16.002" y1="-30.353" x2="-16.764" y2="-37.465" width="0" layer="19" extent="1-1"/>
+<wire x1="-10.414" y1="-18.415" x2="-16.002" y2="-30.353" width="0" layer="19" extent="1-1"/>
+<wire x1="19.05" y1="8.89" x2="-10.414" y2="-18.415" width="0" layer="19" extent="16-16"/>
 </signal>
 <signal name="LED_GREEN">
@@
 <wire x1="-5.334" y1="-8.255" x2="46.99" y2="27.686" width="0" layer="19" extent="1-1"/>
 </signal>
-<signal name="N$14">
-<contactref element="IC2" pad="3"/>
-<contactref element="C9" pad="+"/>
-<wire x1="-10.414" y1="-18.415" x2="-16.002" y2="-30.353" width="0" layer="19" extent="1-1"/>
-</signal>
 <signal name="N$19">
 <contactref element="R8" pad="1"/>
@@
 <wire x1="-17.145" y1="-48.26" x2="-9.525" y2="-52.578" width="0" layer="19" extent="1-1"/>
 </signal>
-<signal name="N$20">
-<contactref element="R7" pad="2"/>
-<contactref element="IC2" pad="2"/>
-<contactref element="C8" pad="+"/>
-<contactref element="C10" pad="1"/>
-<wire x1="-16.764" y1="-37.465" x2="-9.525" y2="-43.942" width="0" layer="19" extent="1-1"/>
-<wire x1="-16.891" y1="-23.622" x2="-16.764" y2="-37.465" width="0" layer="19" extent="1-1"/>
-<wire x1="-12.954" y1="-18.415" x2="-16.891" y2="-23.622" width="0" layer="19" extent="1-1"/>
-</signal>
 <signal name="N$23">
 <contactref element="R7" pad="1"/>
@@
 <wire x1="-14.605" y1="-84.1248" x2="-9.525" y2="-93.98" width="0" layer="19" extent="1-1"/>
 </signal>
+<signal name="N$3">
+<contactref element="C6" pad="2"/>
+<contactref element="JP2" pad="2"/>
+<wire x1="18.669" y1="2.54" x2="-28.575" y2="-90.805" width="0" layer="19" extent="1-1"/>
+</signal>
 </signals>
